Commit message: Adding new main of Jozsef and changed the urdf

File: src/diff_drive_robot/urdf/diff_drive_robot.urdf (robot description, URDF)
Before this commit: robot diff_drive_robot, 4 links, 3 joints
Links:
- removed link caster_wheel
- added link front_caster_wheel, mass 0.01; collision sphere radius=0.02; visual sphere radius=0.02
- added link rear_caster_wheel, mass 0.01; collision sphere radius=0.02; visual sphere radius=0.02
- link base_link: geometry collision cylinder length=0.03 radius=0.17; visual cylinder length=0.03 radius=0.17
- link left_wheel: geometry collision cylinder length=0.02 radius=0.035; visual cylinder length=0.02 radius=0.035
- link right_wheel: geometry collision cylinder length=0.02 radius=0.035; visual cylinder length=0.02 radius=0.035
Joints:
- removed joint caster_wheel_joint
- added joint front_caster_wheel_joint: type fixed, parent base_link, child front_caster_wheel, origin xyz=0.08 0 -0.025 rpy=0 0 0
- added joint rear_caster_wheel_joint: type fixed, parent base_link, child rear_caster_wheel, origin xyz=-0.08 0 -0.025 rpy=0 0 0
- joint left_wheel_joint: origin xyz=-0.1 0.1 0 rpy=0 0 0 -> xyz=0.0 0.11 -0.01 rpy=0 0 0
- joint right_wheel_joint: origin xyz=-0.1 -0.1 0 rpy=0 0 0 -> xyz=0.0 -0.11 -0.01 rpy=0 0 0
